File: hw/c128kbd.kicad_pcb (KiCad board)
At the start: 2 copper layers, 57.2 x 38.1 mm, 29 parts, among them J1 JUMPER2, J2 JUMPER2, P1 USBD+, P2 USBD-, P3 +5V, P4 GND, X1 CONN-25, X2 CONN-3, X3 CONN-6S

Commit message: More or less final version of hardware
Parts:
- removed the P1 at (108.0, 110.5)
- removed the P2 at (111.8, 110.5)
- added C9: 47u 10V, Capacitors_ThroughHole:CP_Radial_D5.0mm_P2.50mm, F.Cu at (114.3, 141.0)
- added R3: 1K*, Resistors_SMD:R_0805_HandSoldering, B.Cu at (114.9, 120.0)
- added X3: CONN-4, Socket_Strips:Socket_Strip_Straight_1x04_Pitch2.54mm, F.Cu at (114.3, 109.2)
- C1, C2, C3, C4: value CAP -> 0.1u
- C10: renamed from C9; value CAP -> 0.1u
- C5, C6: value CAP -> 30p
- C7: value CAPP -> 47u 16V
- C8: value CAP -> 0.1u; footprint Capacitors_ThroughHole:C_Disc_D4.3mm_W1.9mm_P5.00mm -> Capacitors_SMD:C_0805_HandSoldering; moved to B.Cu
- DA1: footprint TO_SOT_Packages_THT:TO-92_Molded_Wide -> TO_SOT_Packages_THT:TO-92_Inline_Wide
- R1: value RES -> 10K; moved to F.Cu
- R2: value RES -> 10K
- R4: renamed from R3; value RES -> 1K*
- X2: value CONN-3 -> CONN-4; footprint Pin_Headers:Pin_Header_Straight_1x03_Pitch2.54mm -> Socket_Strips:Socket_Strip_Straight_1x04_Pitch2.54mm
- moved J1 20.5 mm to (95.9, 118.7), turned to 90 degrees
- moved J2 19.6 mm to (113.7, 127.0), turned to 180 degrees
- moved R1 13.5 mm to (101.6, 119.4), turned to 90 degrees
- moved C1 5.66 mm to (107.9, 138.4), turned to 180 degrees
- moved C10 5.21 mm to (114.3, 138.4), turned to 0 degrees
- moved X2 4.02 mm to (95.2, 109.2)
- moved R4 3.18 mm to (114.9, 121.9), turned to 180 degrees
- moved R2 3.09 mm to (114.3, 116.3)
- moved R5 2.84 mm to (118.1, 130.8)
- moved R6 2.84 mm to (118.1, 128.3)
- moved VD1 2.54 mm to (119.4, 108.0)
- moved VD2 2.54 mm to (124.5, 108.0)
- moved C8 2.52 mm to (123.2, 133.3)
- moved ZQ1 2.01 mm to (108.6, 131.4)
- moved C3 1.80 mm to (101.6, 134.6), turned to 90 degrees
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- renumbered P3 to P1, P4 to P2, R4 to R5, R5 to R6, X3 to X4
Connections:
- J1 pad 1: VCC -> /RSTR
- J1 pad 2: Net-(DD1-Pad44) -> GND
- J2 pad 1: /RSTR -> VCC
- J2 pad 2: GND -> Net-(DD1-Pad44)
- R1 pad 1: GND -> /RSTR
- R1 pad 2: Net-(DD1-Pad44) -> VCC
- R2 pad 1: Net-(R2-Pad1) -> GND
- R2 pad 2: Net-(DD1-Pad39) -> Net-(DD1-Pad44)
- VD1 pad 2: Net-(R2-Pad1) -> Net-(R3-Pad1)
- X2 pad 1: Net-(DD1-Pad30) -> +5V
- X2 pad 2: Net-(DD1-Pad31) -> Net-(DD1-Pad30)
- X2 pad 3: GND -> Net-(DD1-Pad31)
- X4 pad 1: Net-(DD1-Pad2) -> Net-(DD1-Pad3)
- X4 pad 5: Net-(DD1-Pad3) -> Net-(DD1-Pad2)
Routing:
- net GND: track 7.81 -> 198.5 mm
- net +5V: track 64.9 -> 145.0 mm
- net VCC: track 31.1 -> 78.8 mm, vias 1 -> 2
- net Net-(DD1-Pad3): track 0.00 -> 22.9 mm
- net Net-(DD1-Pad2): track 0.00 -> 20.2 mm
- net Net-(R4-Pad1): track 0.00 -> 16.1 mm
- net Net-(DD1-Pad30): track 0.00 -> 15.3 mm
- net Net-(C1-Pad2): track 0.00 -> 13.2 mm
- net Net-(DD1-Pad31): track 0.00 -> 13.0 mm
- net Net-(DD1-Pad33): track 0.00 -> 11.8 mm
- net Net-(C6-Pad2): track 0.00 -> 11.2 mm
- net Net-(DD1-Pad32): track 0.00 -> 11.0 mm
- net Net-(R3-Pad1): track 0.00 -> 10.8 mm
- net Net-(C5-Pad2): track 0.00 -> 8.07 mm
- net Net-(DD1-Pad44): track 2.87 -> 10.5 mm
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Other:
- board size 57.2 x 38.1 mm -> 44.5 x 38.1 mm
- net class Default: via_drill 0.8 -> 0.6

Commit message: Cosmetic fixes
Routing:
- net (no net): track 1.32 -> 0.00 mm
Changed lines of the file:
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@@
     (thickness 1.6)
     (drawings 4)
-    (tracks 436)
+    (tracks 433)
     (zones 0)
     (modules 30)
@@
   )
   (setup
-    (last_trace_width 0.5)
+    (last_trace_width 0.25)
     (user_trace_width 0.5)
     (user_trace_width 0.75)
@@
     (visible_elements FFFFFF7F)
     (pcbplotparams
-      (layerselection 0x0003c_ffffffff)
+      (layerselection 0x0203c_ffffffff)
       (usegerberextensions false)
       (usegerberattributes false)
@@
     (add_net "Net-(C5-Pad2)")
     (add_net "Net-(C6-Pad2)")
-    (add_net "Net-(DD1-Pad1)")
     (add_net "Net-(DD1-Pad2)")
-    (add_net "Net-(DD1-Pad29)")
     (add_net "Net-(DD1-Pad3)")
     (add_net "Net-(DD1-Pad30)")
@@
     (add_net "Net-(DD1-Pad32)")
     (add_net "Net-(DD1-Pad33)")
-    (add_net "Net-(DD1-Pad34)")
-    (add_net "Net-(DD1-Pad37)")
-    (add_net "Net-(DD1-Pad38)")
     (add_net "Net-(DD1-Pad39)")
-    (add_net "Net-(DD1-Pad4)")
     (add_net "Net-(DD1-Pad40)")
     (add_net "Net-(DD1-Pad44)")
     (add_net "Net-(R3-Pad1)")
     (add_net "Net-(R4-Pad1)")
-    (add_net "Net-(X1-Pad2)")
-    (add_net "Net-(X4-Pad2)")
-    (add_net "Net-(X4-Pad6)")
     (add_net VCC)
+  )
+  (module MyLib:Mini_din6 (layer F.Cu)
+    (at 123.19 121.92 90)
+    (tags "MINI DIN")
+    (fp_text reference X4 (at 5.08 -8.89 270) (layer F.SilkS)
+      (effects (font (size 1.524 1.524) (thickness 0.3048)))
+    )
+    (fp_text value CONN-6S (at 0 8.89 90) (layer F.Fab)
+      (effects (font (size 1.524 1.524) (thickness 0.3048)))
+    )
+    (fp_line (start -6.85 7.23) (end -6.85 -5.77) (layer F.SilkS) (width 0.381))
+    (fp_line (start 6.85 7.23) (end -6.85 7.23) (layer F.SilkS) (width 0.381))
+    (fp_line (start 6.85 -5.77) (end 6.85 7.23) (layer F.SilkS) (width 0.381))
+    (fp_line (start -6.85 -5.77) (end 6.85 -5.77) (layer F.SilkS) (width 0.381))
+    (pad S thru_hole rect (at 0 2.54 90) (size 2.2 2.2) (drill 0.70104) (layers *.Cu *.Mask)
+      (net 2 GND))
+    (pad S thru_hole rect (at 1.27 2.54 90) (size 2.2 2.2) (drill 0.70104) (layers *.Cu *.Mask)
+      (net 2 GND))
+    (pad S thru_hole rect (at -1.27 2.54 90) (size 2.2 2.2) (drill 0.70104) (layers *.Cu *.Mask)
+      (net 2 GND))
+    (pad S thru_hole rect (at 6.858 1.778 90) (size 2.2 2.2) (drill 0.70104) (layers *.Cu *.Mask)
+      (net 2 GND))
+    (pad S thru_hole rect (at 6.858 2.794 90) (size 2.2 2.2) (drill 0.70104) (layers *.Cu *.Mask)
+      (net 2 GND))
+    (pad S thru_hole rect (at 6.858 0.762 90) (size 2.2 2.2) (drill 0.70104) (layers *.Cu *.Mask)
+      (net 2 GND))
+    (pad S thru_hole rect (at -6.858 1.778 90) (size 2.2 2.2) (drill 0.70104) (layers *.Cu *.Mask)
+      (net 2 GND))
+    (pad S thru_hole rect (at -6.858 2.794 90) (size 2.2 2.2) (drill 0.70104) (layers *.Cu *.Mask)
+      (net 2 GND))
+    (pad S thru_hole rect (at -6.858 0.762 90) (size 2.2 2.2) (drill 0.70104) (layers *.Cu *.Mask)
+      (net 2 GND))
+    (pad 3 thru_hole circle (at 3.4 -1.25 90) (size 1.6 1.6) (drill 0.9) (layers *.Cu *.Mask)
+      (net 2 GND))
+    (pad 4 thru_hole circle (at -3.4 -1.25 90) (size 1.6 1.6) (drill 0.9) (layers *.Cu *.Mask)
+      (net 1 +5V))
+    (pad 6 thru_hole circle (at -3.4 -3.75 90) (size 1.6 1.6) (drill 0.9) (layers *.Cu *.Mask))
+    (pad 5 thru_hole circle (at 3.4 -3.75 90) (size 1.6 1.6) (drill 0.9) (layers *.Cu *.Mask)
+      (net 5 "Net-(DD1-Pad2)"))
+    (pad 1 thru_hole circle (at 1.3 -1.25 90) (size 1.6 1.6) (drill 0.9) (layers *.Cu *.Mask)
+      (net 6 "Net-(DD1-Pad3)"))
+    (pad 2 thru_hole circle (at -1.3 -1.25 90) (size 1.6 1.6) (drill 0.9) (layers *.Cu *.Mask))
+    (model /home/las/Dropbox/Work/Kicad/3dpackages/minidin_6.wrl
+      (at (xyz 0 0 0))
+      (scale (xyz 1 1 1))
+      (rotate (xyz 0 0 0))
+    )
   )
   (module Capacitors_ThroughHole:CP_Radial_D5.0mm_P2.50mm (layer F.Cu)
@@
     )
   )
-  (module MyLib:Mini_din6 (layer F.Cu)
-    (at 123.19 121.92 90)
-    (tags "MINI DIN")
-    (fp_text reference X4 (at 5.08 -8.89 270) (layer F.SilkS)
-      (effects (font (size 1.524 1.524) (thickness 0.3048)))
-    )
-    (fp_text value CONN-6S (at 0 8.89 90) (layer F.Fab)
-      (effects (font (size 1.524 1.524) (thickness 0.3048)))
-    )
-    (fp_line (start -6.85 -5.77) (end 6.85 -5.77) (layer F.SilkS) (width 0.381))
-    (fp_line (start 6.85 -5.77) (end 6.85 7.23) (layer F.SilkS) (width 0.381))
-    (fp_line (start 6.85 7.23) (end -6.85 7.23) (layer F.SilkS) (width 0.381))
-    (fp_line (start -6.85 7.23) (end -6.85 -5.77) (layer F.SilkS) (width 0.381))
-    (pad 2 thru_hole circle (at -1.3 -1.25 90) (size 1.5 1.5) (drill 0.9) (layers *.Mask B.Cu F.SilkS))
-    (pad 1 thru_hole circle (at 1.3 -1.25 90) (size 1.5 1.5) (drill 0.9) (layers *.Mask B.Cu F.SilkS)
-      (net 6 "Net-(DD1-Pad3)"))
-    (pad 5 thru_hole circle (at 3.4 -3.75 90) (size 1.5 1.5) (drill 0.9) (layers *.Mask B.Cu F.SilkS)
-      (net 5 "Net-(DD1-Pad2)"))
-    (pad 6 thru_hole circle (at -3.4 -3.75 90) (size 1.5 1.5) (drill 0.9) (layers *.Mask B.Cu F.SilkS))
-    (pad 4 thru_hole circle (at -3.4 -1.25 90) (size 1.5 1.5) (drill 0.9) (layers *.Mask B.Cu F.SilkS)
-      (net 1 +5V))
-    (pad 3 thru_hole circle (at 3.4 -1.25 90) (size 1.5 1.5) (drill 0.9) (layers *.Mask B.Cu F.SilkS)
-      (net 2 GND))
-    (pad S thru_hole rect (at -6.858 0.762 90) (size 2.2 2.2) (drill 0.70104) (layers *.Cu *.SilkS *.Mask)
-      (net 2 GND))
-    (pad S thru_hole rect (at -6.858 2.794 90) (size 2.2 2.2) (drill 0.70104) (layers *.Cu *.SilkS *.Mask)
-      (net 2 GND))
-    (pad S thru_hole rect (at -6.858 1.778 90) (size 2.2 2.2) (drill 0.70104) (layers *.Cu *.SilkS *.Mask)
-      (net 2 GND))
-    (pad S thru_hole rect (at 6.858 0.762 90) (size 2.2 2.2) (drill 0.70104) (layers *.Cu *.SilkS *.Mask)
-      (net 2 GND))
-    (pad S thru_hole rect (at 6.858 2.794 90) (size 2.2 2.2) (drill 0.70104) (layers *.Cu *.SilkS *.Mask)
-      (net 2 GND))
-    (pad S thru_hole rect (at 6.858 1.778 90) (size 2.2 2.2) (drill 0.70104) (layers *.Cu *.SilkS *.Mask)
-      (net 2 GND))
-    (pad S thru_hole rect (at -1.27 2.54 90) (size 2.2 2.2) (drill 0.70104) (layers *.Cu *.SilkS *.Mask)
-      (net 2 GND))
-    (pad S thru_hole rect (at 1.27 2.54 90) (size 2.2 2.2) (drill 0.70104) (layers *.Cu *.SilkS *.Mask)
-      (net 2 GND))
-    (pad S thru_hole rect (at 0 2.54 90) (size 2.2 2.2) (drill 0.70104) (layers *.Cu *.SilkS *.Mask)
-      (net 2 GND))
-    (model /home/las/Dropbox/Work/Kicad/3dpackages/minidin_6.wrl
-      (at (xyz 0 0 0))
-      (scale (xyz 1 1 1))
-      (rotate (xyz 0 0 0))
-    )
-  )
   (module Capacitors_ThroughHole:CP_Radial_D5.0mm_P2.50mm (layer F.Cu)
     (at 121.92 135.89)
@@
   (gr_line (start 83.82 143.51) (end 128.27 143.51) (angle 90) (layer Edge.Cuts) (width 0.15))
   (gr_line (start 83.82 105.41) (end 128.27 105.41) (angle 90) (layer Edge.Cuts) (width 0.15))
-  (segment (start 88.9 119.03) (end 88.9 119.38) (width 0.5) (layer F.Cu) (net 0) (status 30))
-  (segment (start 88.9 121.8) (end 89.415 121.8) (width 0.5) (layer F.Cu) (net 0) (status 30))
-  (segment (start 88.9 113.49) (end 89.36 113.49) (width 0.5) (layer F.Cu) (net 0) (status 30))
   (segment (start 121.92 133.39) (end 121.96 133.35) (width 1.5) (layer B.Cu) (net 1))
   (segment (start 121.92 135.89) (end 121.92 133.39) (width 1.5) (layer B.Cu) (net 1))

Commit message: hw: update to kicad 8, should be no problems with cache
Parts:
- DA1: footprint TO_SOT_Packages_THT:TO-92_Inline_Wide -> Package_TO_SOT_THT:TO-92_Inline_Wide
Connections:
- net /40/80 renamed /40/80
- DD1 pad 1: (no net) -> unconnected-(DD1-VBAT-Pad1)
- DD1 pad 29: (no net) -> unconnected-(DD1-PA8-Pad29)
- DD1 pad 34: (no net) -> unconnected-(DD1-PA13-Pad34)
- DD1 pad 37: (no net) -> unconnected-(DD1-PA14-Pad37)
- DD1 pad 38: (no net) -> unconnected-(DD1-PA15-Pad38)
- DD1 pad 4: (no net) -> unconnected-(DD1-PC15-Pad4)
- X1 pad 2: (no net) -> unconnected-(X1-Pad2)
- X4 pad 2: (no net) -> unconnected-(X4-Pad2)
- X4 pad 6: (no net) -> unconnected-(X4-Pad6)
Other:
- net class Default removed
